File: kicad/camera/flash.sch (KiCad schematic (older format))
At the start: 8 parts, among them J2 Conn_01x06, U1 XC6SLX16-FTG256, X1 SG-5032CAN

Commit message: Adding Spartan_ESP scheme
Parts:
- D2: symbol Device:LED -> camera-rescue:LED-Device
- J2: symbol Connector_Generic:Conn_01x06 -> camera-rescue:Conn_01x06-Connector_Generic
- R20, R21, R22, R23: symbol Device:R -> camera-rescue:R-Device
- U1: symbol FPGA_Xilinx_Spartan6:XC6SLX16-FTG256 -> camera-rescue:XC6SLX16-FTG256-FPGA_Xilinx_Spartan6
- X1: symbol Oscillator:SG-5032CAN -> camera-rescue:SG-5032CAN-Oscillator
Changed lines of the file:
@@
 $Descr A4 11693 8268
 encoding utf-8
-Sheet 4 4
+Sheet 4 5
 Title ""
 Date ""
@@
 $EndDescr
 $Comp
-L FPGA_Xilinx_Spartan6:XC6SLX16-FTG256 U1
+L camera-rescue:XC6SLX16-FTG256-FPGA_Xilinx_Spartan6 U1
 U 3 1 60366767
 P 7950 1300
@@
 $EndComp
 $Comp
-L Connector_Generic:Conn_01x06 J2
+L camera-rescue:Conn_01x06-Connector_Generic J2
 U 1 1 6036C970
 P 5900 1250
@@
 	6100 1150 6350 1150
 $Comp
-L power:GND #PWR0144
+L camera-rescue:GND-power #PWR0144
 U 1 1 6037782C
 P 6350 1150
@@
 	6100 1050 6250 1050
 $Comp
-L power:+3V3 #PWR0145
+L camera-rescue:+3V3-power #PWR0145
 U 1 1 60376657
 P 6250 850
@@
 	9700 800  9450 800
 $Comp
-L power:GND #PWR0146
+L camera-rescue:GND-power #PWR0146
 U 1 1 6039DD6C
 P 9600 1600
@@
 NoConn ~ 9450 1800
 $Comp
-L Device:R R?
+L camera-rescue:R-Device R?
 U 1 1 603D29EC
 P 10800 1800
@@
 $EndComp
 $Comp
-L Device:LED D2
+L camera-rescue:LED-Device D2
 U 1 1 603D3617
 P 10800 1400
@@
 $EndComp
 $Comp
-L Device:R R?
+L camera-rescue:R-Device R?
 U 1 1 603D897A
 P 10800 1000
@@
 	10800 1550 10800 1650
 $Comp
-L power:GND #PWR0147
+L camera-rescue:GND-power #PWR0147
 U 1 1 603DB2AE
 P 10800 2150
@@
 	10800 1950 10800 2150
 $Comp
-L power:+3V3 #PWR0148
+L camera-rescue:+3V3-power #PWR0148
 U 1 1 603DCE9C
 P 10800 750
@@
 	10800 1200 10800 1250
 $Comp
-L FPGA_Xilinx_Spartan6:XC6SLX16-FTG256 U1
+L camera-rescue:XC6SLX16-FTG256-FPGA_Xilinx_Spartan6 U1
 U 1 1 60405012
 P 3350 3900
@@
 $EndComp
 $Comp
-L Device:R R?
+L camera-rescue:R-Device R?
 U 1 1 604AAE53
 P 1200 1600
@@
 $EndComp
 $Comp
-L power:GND #PWR0159
+L camera-rescue:GND-power #PWR0159
 U 1 1 604B0CB1
 P 950 1600
@@
 	1050 1600 950  1600
 $Comp
-L Oscillator:SG-5032CAN X?
+L camera-rescue:SG-5032CAN-Oscillator X?
 U 1 1 60606296
 P 7150 3000
@@
 $EndComp
 $Comp
-L power:GND #PWR0160
+L camera-rescue:GND-power #PWR0160
 U 1 1 6060A20D
 P 7150 3500
@@
 SYS_CLK
 $Comp
-L Device:R R?
+L camera-rescue:R-Device R?
 U 1 1 60618459
 P 6800 2850
@@
 $EndComp
 $Comp
-L power:+3V3 #PWR0161
+L camera-rescue:+3V3-power #PWR0161
 U 1 1 6061E4B8
 P 7150 2450
@@
 	1950 800  1950 650
 $Comp
-L power:+3V3 #PWR0162
+L camera-rescue:+3V3-power #PWR0162
 U 1 1 6066CBF3
 P 1950 650
@@
 $EndComp
 $Comp
-L power:+3V3 #PWR0163
+L camera-rescue:+3V3-power #PWR0163
 U 1 1 606706A1
 P 4650 700
