File: kicad/camera/power.sch (KiCad schematic (older format))
At the start: 41 parts, among them J1 Conn_01x02, U1 XC6SLX16-FTG256, U2 NCP1529A, U3 NCP1529A, U4 MP2359

Commit message: Adding Spartan_ESP scheme
Parts:
- C1, C11, C12, C13, C14, C15, C16, C17, C18, C19, C2, C20, C21, C22, C23, C24, C25, C3, C4, C5, C6, C7, C8: symbol Device:C -> camera-rescue:C-Device
- C10, C9: symbol Device:C_Polarized_US -> camera-rescue:C_Polarized_US-Device
- D1: symbol Diode:1N5712 -> camera-rescue:1N5712-Diode
- J1: symbol Connector_Generic:Conn_01x02 -> camera-rescue:Conn_01x02-Connector_Generic
- L1, L2, L3: symbol Device:L -> camera-rescue:L-Device
- R1, R2, R3, R4, R5, R6, R7: symbol Device:R -> camera-rescue:R-Device
- U1: symbol FPGA_Xilinx_Spartan6:XC6SLX16-FTG256 -> camera-rescue:XC6SLX16-FTG256-FPGA_Xilinx_Spartan6
- U2, U3: symbol Regulator_Switching:NCP1529A -> camera-rescue:NCP1529A-Regulator_Switching
- U4: symbol MP2359:MP2359 -> camera-rescue:MP2359-MP2359
