File: kicad/camera/DDR3.sch (KiCad schematic (older format))
At the start: 23 parts, among them U1 XC6SLX16-FTG256, U5 M25P80, U6 MT41K128M16JT-125_IT_K

Commit message: Adding Spartan_ESP scheme
Parts:
- C26, C27, C28, C29, C30, C31, C32, C33: symbol Device:C -> camera-rescue:C-Device
- R10, R11, R12, R13, R14, R15, R16, R17, R18, R19, R8, R9: symbol Device:R -> camera-rescue:R-Device
- U1: symbol FPGA_Xilinx_Spartan6:XC6SLX16-FTG256 -> camera-rescue:XC6SLX16-FTG256-FPGA_Xilinx_Spartan6
- U5: symbol M25P80:M25P80 -> camera-rescue:M25P80-M25P80
- U6: symbol DDR3:MT41K128M16JT-125_IT_K -> camera-rescue:MT41K128M16JT-125_IT_K-DDR3
Other:
- moved on the sheet: C27, R10
Changed lines of the file:
@@
 $Descr A4 11693 8268
 encoding utf-8
-Sheet 3 4
+Sheet 3 5
 Title ""
 Date ""
@@
 $EndDescr
 $Comp
-L FPGA_Xilinx_Spartan6:XC6SLX16-FTG256 U1
+L camera-rescue:XC6SLX16-FTG256-FPGA_Xilinx_Spartan6 U1
 U 2 1 6021A635
 P 3450 4000
@@
 $EndComp
 $Comp
-L Device:C C?
+L camera-rescue:C-Device C?
 U 1 1 60251EEA
 P 5550 7200
@@
 	5550 7000 5550 7050
 $Comp
-L power:GND #PWR0133
+L camera-rescue:GND-power #PWR0133
 U 1 1 60253AD5
 P 5550 7450
@@
 	5550 7450 5550 7350
 $Comp
-L power:+1V5 #PWR0134
+L camera-rescue:+1V5-power #PWR0134
 U 1 1 6026917C
 P 9200 4950
@@
 $EndComp
 $Comp
-L Device:C C?
+L camera-rescue:C-Device C?
 U 1 1 60269ED7
 P 9200 5350
@@
 	9200 5200 9200 5100
 $Comp
-L power:GND #PWR0135
+L camera-rescue:GND-power #PWR0135
 U 1 1 6026D639
 P 9200 5850
@@
 	9200 5500 9200 5850
 $Comp
-L Device:C C?
+L camera-rescue:C-Device C?
 U 1 1 6027007F
 P 9550 5250
@@
 $EndComp
 $Comp
-L Device:C C?
+L camera-rescue:C-Device C?
 U 1 1 602702C0
 P 9550 5550
@@
 $EndComp
 $Comp
-L Device:R R?
+L camera-rescue:R-Device R?
 U 1 1 60278384
 P 9950 5550
@@
 $EndComp
 $Comp
-L Device:R R?
+L camera-rescue:R-Device R?
 U 1 1 60278883
 P 9950 5250
@@
 	9200 5100 9200 4950
 $Comp
-L power:GND #PWR0136
+L camera-rescue:GND-power #PWR0136
 U 1 1 60282F39
 P 9750 5850
@@
 	10550 1700 10550 1650
 $Comp
-L power:GND #PWR0137
+L camera-rescue:GND-power #PWR0137
 U 1 1 602B0704
 P 10550 1700
@@
 	10400 1650 10550 1650
 $Comp
-L Device:C C?
+L camera-rescue:C-Device C?
 U 1 1 602AFC04
 P 10800 1500
@@
 $EndComp
 $Comp
-L Device:C C?
+L camera-rescue:C-Device C?
 U 1 1 602AF1FF
 P 10400 1500
@@
 $EndComp
 $Comp
-L DDR3:MT41K128M16JT-125_IT_K U6
+L camera-rescue:MT41K128M16JT-125_IT_K-DDR3 U6
 U 1 1 6020EC70
 P 9700 2850
+AR Path="/6020EC70" Ref="U6"  Part="1"
+AR Path="/60207289/6020EC70" Ref="U6"  Part="1"
 F 0 "U6" H 9700 4917 50  0000 C CNN
 F 1 "MT41K128M16JT-125_IT_K" H 9700 4826 50  0000 C CNN
@@
 	10450 850  10450 1050
 $Comp
-L power:+1V5 #PWR0138
+L camera-rescue:+1V5-power #PWR0138
 U 1 1 6025A107
 P 10450 850
@@
 Connection ~ 5550 7000
 Wire Wire Line
-	5450 1700 5800 1700
-$Comp
-L Device:R R?
+	5450 1700 5750 1700
+$Comp
+L camera-rescue:R-Device R?
 U 1 1 602D8053
-P 5950 1700
+P 5900 1700
 AR Path="/5FE53EBB/602D8053" Ref="R?"  Part="1"
 AR Path="/60207289/602D8053" Ref="R10"  Part="1"
-F 0 "R10" V 5743 1700 50  0000 C CNN
-F 1 "100" V 5834 1700 50  0000 C CNN
-F 2 "Resistor_SMD:R_0805_2012Metric" V 5880 1700 50  0001 C CNN
-F 3 "~" H 5950 1700 50  0001 C CNN
-F 4 "0.00217" H 5950 1700 50  0001 C CNN "Cost"
-	1    5950 1700
+F 0 "R10" V 5693 1700 50  0000 C CNN
+F 1 "100" V 5784 1700 50  0000 C CNN
+F 2 "Resistor_SMD:R_0805_2012Metric" V 5830 1700 50  0001 C CNN
+F 3 "~" H 5900 1700 50  0001 C CNN
+F 4 "0.00217" H 5900 1700 50  0001 C CNN "Cost"
+	1    5900 1700
 	0    1    1    0
 $EndComp
 $Comp
-L power:GND #PWR0139
+L camera-rescue:GND-power #PWR0139
 U 1 1 602D8D5B
-P 6100 1700
-F 0 "#PWR0139" H 6100 1450 50  0001 C CNN
-F 1 "GND" V 6105 1572 50  0000 R CNN
-F 2 "" H 6100 1700 50  0001 C CNN
-F 3 "" H 6100 1700 50  0001 C CNN
-	1    6100 1700
+P 6050 1700
+F 0 "#PWR0139" H 6050 1450 50  0001 C CNN
+F 1 "GND" V 6055 1572 50  0000 R CNN
+F 2 "" H 6050 1700 50  0001 C CNN
+F 3 "" H 6050 1700 50  0001 C CNN
+	1    6050 1700
 	0    -1   -1   0
 $EndComp
 $Comp
-L Device:C C?
+L camera-rescue:C-Device C?
 U 1 1 602DD3E8
-P 6450 1800
+P 6400 1800
 AR Path="/5FE53EBB/602DD3E8" Ref="C?"  Part="1"
 AR Path="/60207289/602DD3E8" Ref="C27"  Part="1"
-F 0 "C27" V 6198 1800 50  0000 C CNN
-F 1 "100nF" V 6289 1800 50  0000 C CNN
-F 2 "Capacitor_SMD:C_0402_1005Metric" H 6488 1650 50  0001 C CNN
-F 3 "~" H 6450 1800 50  0001 C CNN
-F 4 "0.0062" V 6450 1800 50  0001 C CNN "Cost"
-	1    6450 1800
+F 0 "C27" V 6148 1800 50  0000 C CNN
+F 1 "100nF" V 6239 1800 50  0000 C CNN
+F 2 "Capacitor_SMD:C_0402_1005Metric" H 6438 1650 50  0001 C CNN
+F 3 "~" H 6400 1800 50  0001 C CNN
+F 4 "0.0062" V 6400 1800 50  0001 C CNN "Cost"
+	1    6400 1800
 	0    1    1    0
 $EndComp
 $Comp
-L power:GND #PWR0140
+L camera-rescue:GND-power #PWR0140
 U 1 1 602F4625
-P 6600 1800
-F 0 "#PWR0140" H 6600 1550 50  0001 C CNN
-F 1 "GND" V 6605 1672 50  0000 R CNN
-F 2 "" H 6600 1800 50  0001 C CNN
-F 3 "" H 6600 1800 50  0001 C CNN
-	1    6600 1800
+P 6550 1800
+F 0 "#PWR0140" H 6550 1550 50  0001 C CNN
+F 1 "GND" V 6555 1672 50  0000 R CNN
+F 2 "" H 6550 1800 50  0001 C CNN
+F 3 "" H 6550 1800 50  0001 C CNN
+	1    6550 1800
 	0    -1   -1   0
 $EndComp
-Text Label 5550 1800 0    50   ~ 0
+Text Label 5500 1800 0    50   ~ 0
 DDR_VREF
 Wire Wire Line
-	5450 1800 6300 1800
+	5450 1800 6250 1800
 NoConn ~ 5450 1900
 NoConn ~ 5450 2000
 $Comp
-L Device:R R?
+L camera-rescue:R-Device R?
 U 1 1 6030AD8B
 P 6200 7200
@@
 	6200 7350 6200 7450
 $Comp
-L power:GND #PWR0141
+L camera-rescue:GND-power #PWR0141
 U 1 1 60311984
 P 6200 7450
@@
 $EndComp
 $Comp
-L power:+1V5 #PWR0142
+L camera-rescue:+1V5-power #PWR0142
 U 1 1 6031A221
 P 4850 750
@@
 	2050 900  2150 900
 $Comp
-L power:+3V3 #PWR0143
+L camera-rescue:+3V3-power #PWR0143
 U 1 1 6031FC15
 P 1950 800
@@
 Wire Wire Line
 	1950 800  1950 900
-Text Notes 6600 2350 0    50   ~ 0
+Text Notes 6350 1050 0    50   ~ 0
 TODO:\nConnect DDR, use impedance matching 100R
 Text Label 950  1700 0    50   ~ 0
@@
 	950  5400 1450 5400
 $Comp
-L Device:R R?
+L camera-rescue:R-Device R?
 U 1 1 604F28BC
 P 1200 1800
@@
 	1350 1800 1450 1800
 $Comp
-L power:+3V3 #PWR0149
+L camera-rescue:+3V3-power #PWR0149
 U 1 1 604F5C14
 P 850 1800
@@
 	1050 1800 850  1800
 $Comp
-L Device:R R?
+L camera-rescue:R-Device R?
 U 1 1 6050B63C
 P 1200 5300
@@
 	1350 5300 1450 5300
 $Comp
-L power:+3V3 #PWR0150
+L camera-rescue:+3V3-power #PWR0150
 U 1 1 6050B643
 P 900 5300
@@
 	900  5300 1050 5300
 $Comp
-L M25P80:M25P80 U?
+L camera-rescue:M25P80-M25P80 U?
 U 1 1 60530C0E
 P 7550 5500
@@
 $EndComp
 $Comp
-L power:GND #PWR0151
+L camera-rescue:GND-power #PWR0151
 U 1 1 60547A10
 P 7100 5850
@@
 	7900 5650 8250 5650
 $Comp
-L Device:R R?
+L camera-rescue:R-Device R?
 U 1 1 6054C689
 P 8750 5700
@@
 $EndComp
 $Comp
-L Device:R R?
+L camera-rescue:R-Device R?
 U 1 1 6054CC4C
 P 8750 5400
@@
 Connection ~ 8750 5550
 $Comp
-L Device:R R?
+L camera-rescue:R-Device R?
 U 1 1 6054D055
 P 8150 5450
@@
 	8000 5450 7900 5450
 $Comp
-L power:+3V3 #PWR0152
+L camera-rescue:+3V3-power #PWR0152
 U 1 1 605508C0
 P 8350 5450
@@
 	7900 5550 8750 5550
 $Comp
-L power:+3V3 #PWR0153
+L camera-rescue:+3V3-power #PWR0153
 U 1 1 6055A827
 P 7950 4950
@@
 	7950 5350 7900 5350
 $Comp
-L Device:C C?
+L camera-rescue:C-Device C?
 U 1 1 6055C08B
 P 8150 5100
@@
 $EndComp
 $Comp
-L power:GND #PWR0154
+L camera-rescue:GND-power #PWR0154
 U 1 1 6055CC40
 P 8450 5150
@@
 	7950 5100 7950 5350
 $Comp
-L power:GND #PWR0155
+L camera-rescue:GND-power #PWR0155
 U 1 1 605645A3
 P 8750 5900
@@
 	8750 5900 8750 5850
 $Comp
-L power:+3V3 #PWR0156
+L camera-rescue:+3V3-power #PWR0156
 U 1 1 60565CEA
 P 8750 5200
@@
 FPGA_CSO_B
 $Comp
-L power:+3V3 #PWR0157
+L camera-rescue:+3V3-power #PWR0157
 U 1 1 60574E13
 P 6350 5350
@@
 $EndComp
 $Comp
-L Device:R R?
+L camera-rescue:R-Device R?
 U 1 1 605799DC
 P 6950 5450
@@
 FPGA_MISO
 $Comp
-L power:+3V3 #PWR0158
+L camera-rescue:+3V3-power #PWR0158
 U 1 1 60587D66
 P 6350 5550
@@
 	6400 5550 6350 5550
 $Comp
-L Device:R R?
+L camera-rescue:R-Device R?
 U 1 1 6058B015
 P 6550 5550
@@
 	7200 5350 6700 5350
 $Comp
-L Device:R R?
+L camera-rescue:R-Device R?
 U 1 1 6056DADD
 P 6550 5350

Commit message: ESP_LAN
Parts:
- added R?: 4.7k, Resistor_SMD:R_0805_2012Metric, symbol camera-rescue:R-Device
Changed lines of the file:
@@
+	0    1    1    0
+$EndComp
+$Comp
+L camera-rescue:R-Device R?
+U 1 1 5FE9180F
+P 4050 5050
+AR Path="/5FE53EBB/5FE9180F" Ref="R?"  Part="1"
+AR Path="/60207289/5FE9180F" Ref="R?"  Part="1"
+F 0 "R?" V 3843 5050 50  0000 C CNN
+F 1 "4.7k" V 3934 5050 50  0000 C CNN
+F 2 "Resistor_SMD:R_0805_2012Metric" V 3980 5050 50  0001 C CNN
+F 3 "~" H 4050 5050 50  0001 C CNN
+F 4 "0.00217" H 4050 5050 50  0001 C CNN "Cost"
+	1    4050 5050
 	0    1    1    0
 $EndComp
