File: kicad/camera/ESP.sch (KiCad schematic (older format))
At the start: 0 parts

Commit message: ESP_LAN
Parts:
- added C? (x8): 100nF, Capacitor_SMD:C_0402_1005Metric, symbol camera-rescue:C-Device
- added C? (x2): 10nF, Capacitor_SMD:C_0402_1005Metric, symbol camera-rescue:C-Device
- added C?: 22nF, Capacitor_SMD:C_0402_1005Metric, symbol camera-rescue:C-Device
- added C?: 1uF, Capacitor_SMD:C_0402_1005Metric, symbol camera-rescue:C-Device
- added C?: 270pF, Capacitor_SMD:C_0402_1005Metric, symbol camera-rescue:C-Device
- added FB?: 30R, symbol Device:Ferrite_Bead
- added J?: RJ45_Abracon_ARJP11A-MASA-B-A-EMU2, Connector_RJ:RJ45_Abracon_ARJP11A-MA_Horizontal, symbol Connector:RJ45_Abracon_ARJP11A-MASA-B-A-EMU2
- added R? (x2): 330, Resistor_SMD:R_0805_2012Metric, symbol camera-rescue:R-Device
- added R?: 12.1k, Resistor_SMD:R_0805_2012Metric, symbol camera-rescue:R-Device
- added R? (x3): 33, Resistor_SMD:R_0805_2012Metric, symbol camera-rescue:R-Device
- added R?: 10k, Resistor_SMD:R_0805_2012Metric, symbol camera-rescue:R-Device
- added R?: 4.7k, Resistor_SMD:R_0805_2012Metric, symbol camera-rescue:R-Device
- added R? (x4): 10R, Resistor_SMD:R_0805_2012Metric, symbol camera-rescue:R-Device
- added R?: 1.5k, Resistor_SMD:R_0805_2012Metric, symbol camera-rescue:R-Device
- added R? (x4): 49.9, Resistor_SMD:R_0805_2012Metric, symbol camera-rescue:R-Device
- added R?: 0R, Resistor_SMD:R_0805_2012Metric, symbol camera-rescue:R-Device
- added U?: ESP32-WROOM-32, RF_Module:ESP32-WROOM-32, symbol RF_Module:ESP32-WROOM-32
- added U?: LAN8720A, Package_DFN_QFN:QFN-24-1EP_4x4mm_P0.5mm_EP2.6x2.6mm, symbol Interface_Ethernet:LAN8720A
- added X?: SG-5032CAN-Oscillator, Oscillator:Oscillator_SMD_SeikoEpson_SG8002LB-4Pin_5.0x3.2mm, symbol camera-rescue:SG-5032CAN-Oscillator
Connections:
- new net: C?.1, C?.1, C?.1, C?.1, FB?.1, U?.1 (VDD2A), U?.19 (VDD1A)
- new net: R?.1, U?.10 (RXER/PHYAD0)
- new net: R?.1, U?.11 (CRS_DV/MODE2)
- new net: R?.2, U?.14 (INT/REFCLKO)
- new net: C?.2, R?.1, U?.15 (RST)
- new net: R?.2, U?.2 (LED2/nINTSEL)
- new net: J?.2 (TD-), R?.1, U?.20 (TXN)
- new net: J?.1 (TD+), R?.1, U?.21 (TXP)
- new net: J?.6 (RD-), R?.1, U?.22 (RXN)
- new net: J?.3 (RD+), R?.1, U?.23 (RXP)
- new net: R?.2, U?.24 (RBIAS)
- new net: R?.2, U?.3 (LED1/REGOFF)
- new net: R?.1, U?.5 (XTAL1/CLKIN)
- new net: C?.1, C?.1, U?.6 (VDDCR)
- new net: R?.1, U?.7 (RXD1/MODE1)
- new net: R?.1, U?.8 (RXD0/MODE0)
- new net: J?.12 (LLED-), R?.1
- new net: J?.14 (RLED-), R?.1
- new net: J?.15 (SHIELD), R?.2
- new net: R?.1, R?.2, X?.3 (OUT)
- new net +12V: J?.9 (V+)
- new net +3V3: C?.1, C?.1, C?.1, C?.1, C?.1, C?.2, FB?.2, J?.11 (LLED+), J?.13 (RLED+), J?.4 (CT), J?.5 (CT), R?.2, R?.2, R?.2, R?.2, R?.2, R?.2, R?.2, U?.2 (VDD), U?.3 (EN), U?.9 (VDDIO), X?.4 (VCC)
- new net ETH_CRS_DV: R?.2
- new net ETH_MDC: U?.13 (MDC)
- new net ETH_MDIO: R?.1, U?.12 (MDIO)
- new net ETH_REFLCK: R?.1, R?.2
- new net ETH_RXD0: R?.2
- new net ETH_RXD1: R?.2
- new net ETH_TXD0: U?.17 (TXD0)
- new net ETH_TXD1: U?.18 (TXD1)
- new net ETH_TXDEN: U?.16 (TXEN)
- new net GND: C?.1, C?.1, C?.2, C?.2, C?.2, C?.2, C?.2, C?.2, C?.2, C?.2, C?.2, C?.2, C?.2, J?.10 (V-), R?.1, R?.1, R?.1, U?.1 (GND), U?.15 (GND), U?.25 (VSS), U?.38 (GND), U?.39 (GND), X?.2 (GND)
- new net PHY_PWR: R?.2, X?.1 (~ST)
- no-connect marks 0 -> 1
